Commit message: Tf2 and observer working with ros2bag

File: yf_description/urdf/components/asv_gps.xacro (robot description, xacro)
@@ -22,10 +22,10 @@
     <joint name="gps_joint" type="fixed">
       <origin
-        xyz="-0.27 -0.28 0.54"
+        xyz="0.27 0.28 -0.54"
         rpy="0 0 0" />
       <parent
+        link="gps_link" />
+      <child
         link="base_link" />
-      <child
-        link="gps_link" />
     </joint>
   </xacro:macro>
