Commit message: new tf broadcast with neihbor

File: yf_description/urdf/asv_loyola.urdf.xacro (robot description, xacro)
@@ -1,11 +1,20 @@
 <?xml version="1.0"?>
 <robot name="asv_loyola" xmlns:xacro="http://www.ros.org/wiki/xacro">
+  <xacro:arg name="id" default="0" />
+  <xacro:arg name="own" default="false"/>
   <!-- Include dynamics macros -->
   <xacro:include filename="$(find yf_description)/urdf/components/asv_gps.xacro"/>
   <xacro:include filename="$(find yf_description)/urdf/components/asv_camera.xacro"/>
   <xacro:include filename="$(find yf_description)/urdf/components/asv_imu.xacro"/>
-  <xacro:include filename="base_asv.xacro" />
-  <xacro:asv_camera/>
-  <xacro:asv_gps/>
-  <xacro:asv_imu/>
+  <xacro:include filename="base_asv.xacro"/>
+  <xacro:include filename="base_neighbor.xacro"/>
+  <xacro:if value="$(arg own)">
+    <xacro:base_asv/>
+    <xacro:asv_camera/>
+    <xacro:asv_gps/>
+    <xacro:asv_imu/>
+  </xacro:if>
+  <xacro:unless value="$(arg own)">
+    <xacro:base_asv_neighbor name="ASV$(arg id)"/>
+  </xacro:unless>
 </robot>

File: yf_description/urdf/base_asv.xacro (robot description, xacro)
@@ -1,152 +1,154 @@
 <?xml version="1.0"?>
 <robot xmlns:xacro="http://www.ros.org/wiki/xacro">
-  <link
-    name="base_link">
-    <visual>
-      <origin
-        xyz="0 0 0"
-        rpy="0 0 ${pi/2}" />
-      <geometry>
-        <mesh
-          filename="package://asv_description/meshes/base_link.STL" />
-      </geometry>
-      <material
-        name="">
-        <color
-          rgba="1 1 0 1" />
-      </material>
-    </visual>
-    <visual name="join_right_gps">
-      <origin xyz="-0.225 -0.25  0.28" rpy="0.0 0.0 0.0" />
-      <geometry>
-        <box size="0.03 0.03 0.50" />
-      </geometry>
-      <material
+  <xacro:macro name="base_asv">
+    <link
+      name="base_link">
+      <visual>
+        <origin
+          xyz="0 0 0"
+          rpy="0 0 ${pi/2}" />
+        <geometry>
+          <mesh
+            filename="package://yf_description/meshes/base_link.STL" />
+        </geometry>
+        <material
           name="">
           <color
-            rgba="0.89 0.895 0.90 1" />
+            rgba="1 1 0 1" />
         </material>
-    </visual>
-    <visual name="join_left_gps">
-      <origin xyz="-0.225 0.25 0.28" rpy="0.0 0.0 0.0" />
-      <geometry>
-        <box size="0.03 0.03 0.50" />
-      </geometry>
-      <material
+      </visual>
+      <visual name="join_right_gps">
+        <origin xyz="-0.225 -0.25  0.28" rpy="0.0 0.0 0.0" />
+        <geometry>
+          <box size="0.03 0.03 0.50" />
+        </geometry>
+        <material
+            name="">
+            <color
+              rgba="0.89 0.895 0.90 1" />
+          </material>
+      </visual>
+      <visual name="join_left_gps">
+        <origin xyz="-0.225 0.25 0.28" rpy="0.0 0.0 0.0" />
+        <geometry>
+          <box size="0.03 0.03 0.50" />
+        </geometry>
+        <material
+            name="">
+            <color
+              rgba="0.89 0.895 0.90 1" />
+          </material>
+      </visual>
+      <visual name="join_top_gps">
+        <origin xyz="-0.225 0.0 0.4" rpy="0.0 0.0 0.0" />
+        <geometry>
+          <box size="0.03 0.51 0.03" />
+        </geometry>
+        <material
+            name="">
+            <color
+              rgba="0.89 0.895 0.90 1" />
+          </material>
+      </visual>
+      <collision>
+        <origin
+          xyz="0 0 0"
+          rpy="0 0 ${pi/2}" />
+        <geometry>
+          <mesh
+            filename="package://yf_description/meshes/base_link.STL" />
+        </geometry>
+      </collision>
+    </link>
+    <link
+      name="Motor_izquierda_link">
+      <visual>
+        <origin
+          xyz="0 0 0"
+          rpy="0 0 0" />
+        <geometry>
+          <mesh
+            filename="package://yf_description/meshes/Motor_izquierda_link.STL" />
+        </geometry>
+        <material
           name="">
           <color
-            rgba="0.89 0.895 0.90 1" />
+            rgba="0 0 0 1" />
         </material>
-    </visual>
-    <visual name="join_top_gps">
-      <origin xyz="-0.225 0.0 0.4" rpy="0.0 0.0 0.0" />
-      <geometry>
-        <box size="0.03 0.51 0.03" />
-      </geometry>
-      <material
+      </visual>
+      <collision>
+        <origin
+          xyz="0 0 0"
+          rpy="0 0 0" />
+        <geometry>
+          <mesh
+            filename="package://yf_description/meshes/Motor_izquierda_link.STL" />
+        </geometry>
+      </collision>
+    </link>
+    <link
+      name="Motor_derecha_link">
+      <visual>
+        <origin
+          xyz="0 0 0"
+          rpy="0 0 0" />
+        <geometry>
+          <mesh
+            filename="package://yf_description/meshes/Motor_derecha_link.STL" />
+        </geometry>
+        <material
           name="">
           <color
-            rgba="0.89 0.895 0.90 1" />
+            rgba="0 0 0 1" />
         </material>
-    </visual>
-    <collision>
+      </visual>
+      <collision>
+        <origin
+          xyz="0 0 0"
+          rpy="0 0 0" />
+        <geometry>
+          <mesh
+            filename="package://yf_description/meshes/Motor_derecha_link.STL" />
+        </geometry>
+      </collision>
+    </link>
+    <joint
+      name="left_motor_joint"
+      type="fixed">
       <origin
-        xyz="0 0 0"
-        rpy="0 0 ${pi/2}" />
-      <geometry>
-        <mesh
-          filename="package://asv_description/meshes/base_link.STL" />
-      </geometry>
-    </collision>
-  </link>
-  <link
-    name="Motor_izquierda_link">
-    <visual>
-      <origin
-        xyz="0 0 0"
-        rpy="0 0 0" />
-      <geometry>
-        <mesh
-          filename="package://asv_description/meshes/Motor_izquierda_link.STL" />
-      </geometry>
-      <material
-        name="">
-        <color
-          rgba="0 0 0 1" />
-      </material>
-    </visual>
-    <collision>
-      <origin
-        xyz="0 0 0"
-        rpy="0 0 0" />
-      <geometry>
-        <mesh
-          filename="package://asv_description/meshes/Motor_izquierda_link.STL" />
-      </geometry>
-    </collision>
-  </link>
-  <link
-    name="Motor_derecha_link">
-    <visual>
-      <origin
-        xyz="0 0 0"
-        rpy="0 0 0" />
-      <geometry>
-        <mesh
-          filename="package://asv_description/meshes/Motor_derecha_link.STL" />
-      </geometry>
-      <material
-        name="">
-        <color
-          rgba="0 0 0 1" />
-      </material>
-    </visual>
-    <collision>
-      <origin
-        xyz="0 0 0"
-        rpy="0 0 0" />
-      <geometry>
-        <mesh
-          filename="package://asv_description/meshes/Motor_derecha_link.STL" />
-      </geometry>
-    </collision>
-  </link>
-  <joint
-    name="left_motor_joint"
-    type="fixed">
-    <origin
-      xyz="-0.44372 0.3375 -0.20667"
-      rpy="-1.5708 0.0 -1.5708" />
-    <parent
-      link="base_link" />
-    <child
-      link="Motor_izquierda_link" />
-    <axis
-      xyz="0 0 1" />
-    <limit
-      effort="100"
-      velocity="100" />
-    <dynamics
-      damping="0.1"
-      friction="0.1" />
-  </joint>
- <joint
-    name="right_motor_joint"
-        type="fixed">
-        <origin
-        xyz="-0.44372 -0.3375 -0.20667"
+        xyz="-0.44372 0.3375 -0.20667"
         rpy="-1.5708 0.0 -1.5708" />
-        <parent
+      <parent
         link="base_link" />
-        <child
-        link="Motor_derecha_link" />
-        <axis
+      <child
+        link="Motor_izquierda_link" />
+      <axis
         xyz="0 0 1" />
-        <limit
+      <limit
         effort="100"
         velocity="100" />
-        <dynamics
+      <dynamics
         damping="0.1"
         friction="0.1" />
     </joint>
+  <joint
+      name="right_motor_joint"
+          type="fixed">
+          <origin
+          xyz="-0.44372 -0.3375 -0.20667"
+          rpy="-1.5708 0.0 -1.5708" />
+          <parent
+          link="base_link" />
+          <child
+          link="Motor_derecha_link" />
+          <axis
+          xyz="0 0 1" />
+          <limit
+          effort="100"
+          velocity="100" />
+          <dynamics
+          damping="0.1"
+          friction="0.1" />
+      </joint>
+  </xacro:macro>
 </robot>

Commit message: New topic-based structure based on multiple ASVs, and reorganization of nodes and packages

File: yf_description/urdf/asv_loyola.urdf.xacro (robot description, xacro)
@@ -10,8 +10,8 @@
   <xacro:include filename="base_neighbor.xacro"/>
   <xacro:if value="$(arg own)">
-    <xacro:base_asv/>
-    <xacro:asv_camera/>
-    <xacro:asv_gps/>
-    <xacro:asv_imu/>
+    <xacro:base_asv name="ASV$(arg id)"/>
+    <xacro:asv_camera name="ASV$(arg id)"/>
+    <xacro:asv_gps name="ASV$(arg id)"/>
+    <xacro:asv_imu name="ASV$(arg id)"/>
   </xacro:if>
   <xacro:unless value="$(arg own)">

File: yf_description/urdf/base_asv.xacro (robot description, xacro)
@@ -1,7 +1,7 @@
 <?xml version="1.0"?>
 <robot xmlns:xacro="http://www.ros.org/wiki/xacro">
-  <xacro:macro name="base_asv">
+  <xacro:macro name="base_asv" params="name">
     <link
-      name="base_link">
+      name="${name}/base_link">
       <visual>
         <origin
@@ -62,5 +62,5 @@
     </link>
     <link
-      name="Motor_izquierda_link">
+      name="${name}/Motor_izquierda_link">
       <visual>
         <origin
@@ -88,5 +88,5 @@
     </link>
     <link
-      name="Motor_derecha_link">
+      name="${name}/Motor_derecha_link">
       <visual>
         <origin
@@ -114,5 +114,5 @@
     </link>
     <joint
-      name="left_motor_joint"
+      name="${name}/left_motor_joint"
       type="fixed">
       <origin
@@ -120,7 +120,7 @@
         rpy="-1.5708 0.0 -1.5708" />
       <parent
-        link="base_link" />
+        link="${name}/base_link" />
       <child
-        link="Motor_izquierda_link" />
+        link="${name}/Motor_izquierda_link" />
       <axis
         xyz="0 0 1" />
@@ -133,5 +133,5 @@
     </joint>
   <joint
-      name="right_motor_joint"
+      name="${name}/right_motor_joint"
           type="fixed">
           <origin
@@ -139,7 +139,7 @@
           rpy="-1.5708 0.0 -1.5708" />
           <parent
-          link="base_link" />
+          link="${name}/base_link" />
           <child
-          link="Motor_derecha_link" />
+          link="${name}/Motor_derecha_link" />
           <axis
           xyz="0 0 1" />

File: yf_description/urdf/base_neighbor.xacro (robot description, xacro)
@@ -3,5 +3,5 @@
   <xacro:macro name="base_asv_neighbor" params="name">
     <link
-      name="${name}">
+      name="${name}/base_link">
       <visual>
         <origin
@@ -62,5 +62,5 @@
     </link>
     <link
-      name="${name}_Motor_izquierda_link">
+      name="${name}/Motor_izquierda_link">
       <visual>
         <origin
@@ -88,5 +88,5 @@
     </link>
     <link
-      name="${name}_Motor_derecha_link">
+      name="${name}/Motor_derecha_link">
       <visual>
         <origin
@@ -114,5 +114,5 @@
     </link>
     <joint
-      name="${name}_left_motor_joint"
+      name="${name}/left_motor_joint"
       type="fixed">
       <origin
@@ -120,7 +120,7 @@
         rpy="-1.5708 0.0 -1.5708" />
       <parent
-        link="${name}" />
+        link="${name}/base_link" />
       <child
-        link="${name}_Motor_izquierda_link" />
+        link="${name}/Motor_izquierda_link" />
       <axis
         xyz="0 0 1" />
@@ -133,5 +133,5 @@
     </joint>
   <joint
-      name="${name}_right_motor_joint"
+      name="${name}/right_motor_joint"
           type="fixed">
           <origin
@@ -139,7 +139,7 @@
           rpy="-1.5708 0.0 -1.5708" />
           <parent
-          link="${name}" />
+          link="${name}/base_link"/>
           <child
-          link="${name}_Motor_derecha_link" />
+          link="${name}/Motor_derecha_link" />
           <axis
           xyz="0 0 1" />

File: yf_description/urdf/components/asv_camera.xacro (robot description, xacro)
@@ -1,7 +1,7 @@
 <?xml version="1.0" encoding="UTF-8"?>
 <robot xmlns:xacro="http://ros.org/wiki/xacro">
-  <xacro:macro name="asv_camera">
+  <xacro:macro name="asv_camera" params="name">
     <link
-      name="asv_camera">
+      name="${name}/asv_camera">
       <visual>
         <origin
@@ -22,5 +22,5 @@
     </link>
     <joint
-      name="camera_joint"
+      name="${name}/camera_joint"
       type="fixed">
       <origin
@@ -28,17 +28,17 @@
         rpy="0.0 0.0 0.0" />
       <parent
-        link="base_link" />
+        link="${name}/base_link" />
       <child
-        link="asv_camera"/>
+        link="${name}/asv_camera"/>
     </joint>
-    <link name="camera_link_optical">
+    <link name="${name}/camera_link_optical">
     </link>
-    <joint name="camera_optical_joint" type="fixed">
+    <joint name="${name}/camera_optical_joint" type="fixed">
         <!-- these values have to be these values otherwise the gazebo camera
             image won't be aligned properly with the frame it is supposedly
             originating from -->
         <origin xyz="0 0 0" rpy="${pi/2} ${pi} ${pi/2}"/>
-        <parent link="asv_camera"/>
-        <child link="camera_link_optical"/>
+        <parent link="${name}/asv_camera"/>
+        <child link="${name}/camera_link_optical"/>
     </joint>
   </xacro:macro>

File: yf_description/urdf/components/asv_gps.xacro (robot description, xacro)
@@ -1,6 +1,6 @@
 <?xml version="1.0" encoding="UTF-8"?>
 <robot xmlns:xacro="http://ros.org/wiki/xacro">
-  <xacro:macro name="asv_gps">
-    <link name="gps_link">
+  <xacro:macro name="asv_gps" params="name">
+    <link name="${name}/gps_link">
       <visual>
         <geometry>
@@ -20,12 +20,12 @@
       </collision>
     </link>
-    <joint name="gps_joint" type="fixed">
+    <joint name="${name}/gps_joint" type="fixed">
       <origin
         xyz="0.27 0.28 -0.54"
         rpy="0 0 0" />
       <parent
-        link="gps_link" />
+        link="${name}/gps_link" />
       <child
-        link="base_link" />
+        link="${name}/base_link" />
     </joint>
   </xacro:macro>

File: yf_description/urdf/components/asv_imu.xacro (robot description, xacro)
@@ -1,6 +1,6 @@
 <?xml version="1.0"?>
 <robot xmlns:xacro="http://ros.org/wiki/xacro">
-  <xacro:macro name="asv_imu">
-    <link name="imu_link">
+  <xacro:macro name="asv_imu" params="name">
+    <link name="${name}/imu_link">
       <visual>
         <geometry>
@@ -19,8 +19,8 @@
       </collision>
     </link>
-    <joint name="imu_joint" type="fixed">
+    <joint name="${name}/imu_joint" type="fixed">
       <origin xyz="0 0 0.14" rpy="0 0 0"/>
-      <parent link="base_link"/>
-      <child link="imu_link"/>
+      <parent link="${name}/base_link"/>
+      <child link="${name}/imu_link"/>
     </joint>
   </xacro:macro>
